File: Reference-designs/Attiny-2313/B-timer/B-timer.kicad_pcb (KiCad board)
At the start: 2 copper layers, 41.7 x 31.6 mm, 104 parts, among them SW1 SW_Push, SW2 SW_Push, SW3 SW_Push, U2 ATTINY2313-20MU

Commit message: Update version
Parts:
- removed U2: ATTINY2313-20MU, Bitraf:VQFN20-SMALL
- added BZ1: Buzzer, Buzzers_Beepers:Buzzer_Murata_PKMCS0909E4000-R1, F.Cu at (189.1, 88.8)
- added J2: Conn_02x03_Odd_Even, Pin_Headers:Pin_Header_Straight_2x03_Pitch2.54mm_SMD, F.Cu at (178.1, 71.2)
- added U1: ATTINY2313-20MU, Bitraf:VQFN20-SMALL, F.Cu at (209.0, 102.2)
- D1, D10, D11, D12, D13, D14, D15, D16, D17, D18, D19, D2, D20, D21, D22, D23, D24, D25, D26, D27, D28, D29, D3, D30, D31, D32, D33, D34, D35, D36, D37, D38, D39, D4, D40, D41, D42, D43, D44, D45, D46, D47, D48, D49, D5, D50, D51, D52, D53, D54, D55, D56, D57, D58, D59, D6, D60, D61, D62, D63, D64, D65, D66, D67, D68, D69, D7, D70, D71, D72, D73, D74, D75, D76, D77, D78, D79, D8, D80, D81, D82, D83, D84, D85, D86, D87, D88, D89, D9, D90: footprint Bitraf:LED_0402 -> LEDs:LED_0603
- R1, R10, R2, R3, R4, R5, R6, R7, R8, R9: footprint Bitraf:R_0402 -> Resistors_SMD:R_0402
- SW1, SW2, SW3: footprint Bitraf:PTS_540 -> Buttons_Switches_SMD:SW_SPST_B3S-1000
- moved D42 71.7 mm to (152.3, 73.3)
- moved D51 71.7 mm to (152.3, 74.7)
- moved D54 65.9 mm to (152.3, 78.7)
- moved D49 63.6 mm to (149.3, 76.0)
- moved D55 63.5 mm to (146.8, 80.1)
- moved D67 61.7 mm to (152.3, 76.0)
- moved SW3 59.8 mm to (182.4, 116.0)
- moved D57 58.7 mm to (133.4, 92.2)
- moved D53 58.7 mm to (139.3, 94.3)
- moved D69 57.9 mm to (146.8, 81.4)
- moved D48 57.3 mm to (140.9, 83.5)
- moved D50 55.7 mm to (143.9, 80.8)
- moved D56 55.1 mm to (138.0, 87.5)
- moved D83 54.5 mm to (146.8, 85.5)
- moved D52 53.4 mm to (143.9, 82.1)
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Connections:
- D1 pad 1: D7 -> D0
- D10 pad 1: D0 -> D1
- D11 pad 2: Net-(D10-Pad2) -> Net-(D11-Pad2)
- D12 pad 1: D2 -> D1
- D13 pad 1: D3 -> D1
- D13 pad 2: Net-(D12-Pad2) -> Net-(D13-Pad2)
- D14 pad 1: D4 -> D1
- D14 pad 2: Net-(D12-Pad2) -> Net-(D14-Pad2)
- D15 pad 1: D5 -> D1
- D15 pad 2: Net-(D12-Pad2) -> Net-(D15-Pad2)
- D16 pad 1: D6 -> D1
- D16 pad 2: Net-(D12-Pad2) -> Net-(D16-Pad2)
- D18 pad 1: D0 -> D1
- D19 pad 1: D1 -> D2
- D19 pad 2: Net-(D18-Pad2) -> Net-(D10-Pad2)
- D2 pad 2: Net-(D12-Pad2) -> Net-(D11-Pad2)
- D20 pad 2: Net-(D18-Pad2) -> Net-(D1-Pad2)
- D21 pad 1: D3 -> D2
- D21 pad 2: Net-(D10-Pad2) -> Net-(D12-Pad2)
- D22 pad 1: D4 -> D2
- D22 pad 2: Net-(D10-Pad2) -> Net-(D13-Pad2)
- D23 pad 1: D5 -> D2
- D23 pad 2: Net-(D10-Pad2) -> Net-(D14-Pad2)
- D24 pad 1: D6 -> D2
- D24 pad 2: Net-(D10-Pad2) -> Net-(D15-Pad2)
- D25 pad 2: Net-(D17-Pad2) -> Net-(D16-Pad2)
- D26 pad 1: D0 -> D2
- D26 pad 2: Net-(D26-Pad2) -> Net-(D17-Pad2)
- D27 pad 1: D1 -> D2
- D27 pad 2: Net-(D26-Pad2) -> Net-(D18-Pad2)
- D28 pad 1: D2 -> D3
- D28 pad 2: Net-(D26-Pad2) -> Net-(D10-Pad2)
- D29 pad 2: Net-(D26-Pad2) -> Net-(D1-Pad2)
- D3 pad 1: D1 -> D0
- D3 pad 2: Net-(D1-Pad2) -> Net-(D12-Pad2)
- D30 pad 1: D4 -> D3
- D30 pad 2: Net-(D18-Pad2) -> Net-(D11-Pad2)
- D31 pad 1: D5 -> D3
- D31 pad 2: Net-(D18-Pad2) -> Net-(D13-Pad2)
- D32 pad 1: D6 -> D3
- D32 pad 2: Net-(D18-Pad2) -> Net-(D14-Pad2)
- D33 pad 2: Net-(D17-Pad2) -> Net-(D15-Pad2)
- D34 pad 1: D0 -> D3
- D34 pad 2: Net-(D34-Pad2) -> Net-(D16-Pad2)
- D35 pad 1: D1 -> D3
- D35 pad 2: Net-(D34-Pad2) -> Net-(D17-Pad2)
- D36 pad 1: D2 -> D3
- D36 pad 2: Net-(D34-Pad2) -> Net-(D18-Pad2)
- D37 pad 1: D3 -> D4
- D37 pad 2: Net-(D34-Pad2) -> Net-(D10-Pad2)
- D38 pad 2: Net-(D34-Pad2) -> Net-(D1-Pad2)
- D39 pad 1: D5 -> D4
- D39 pad 2: Net-(D26-Pad2) -> Net-(D11-Pad2)
- D4 pad 1: D2 -> D0
- D4 pad 2: Net-(D1-Pad2) -> Net-(D13-Pad2)
- D40 pad 1: D6 -> D4
- D40 pad 2: Net-(D26-Pad2) -> Net-(D12-Pad2)
- D41 pad 2: Net-(D17-Pad2) -> Net-(D14-Pad2)
- D42 pad 1: D8 -> D4
- D42 pad 2: Net-(D1-Pad2) -> Net-(D15-Pad2)
- D43 pad 1: D0 -> D4
- D43 pad 2: Net-(D43-Pad2) -> Net-(D16-Pad2)
- D44 pad 1: D1 -> D4
- D44 pad 2: Net-(D43-Pad2) -> Net-(D17-Pad2)
- D45 pad 1: D2 -> D4
- D45 pad 2: Net-(D43-Pad2) -> Net-(D18-Pad2)
- D46 pad 1: D3 -> D5
- D46 pad 2: Net-(D43-Pad2) -> Net-(D10-Pad2)
- D47 pad 1: D4 -> D5
- D47 pad 2: Net-(D43-Pad2) -> Net-(D1-Pad2)
- D48 pad 1: D9 -> D5
- D48 pad 2: Net-(D1-Pad2) -> Net-(D11-Pad2)
- D49 pad 1: D7 -> D5
- D5 pad 1: D3 -> D0
- D5 pad 2: Net-(D1-Pad2) -> Net-(D14-Pad2)
- D50 pad 1: D8 -> D5
- D50 pad 2: Net-(D12-Pad2) -> Net-(D13-Pad2)
- D51 pad 1: D9 -> D5
- D51 pad 2: Net-(D12-Pad2) -> Net-(D15-Pad2)
- D52 pad 1: D7 -> D5
- D52 pad 2: Net-(D10-Pad2) -> Net-(D16-Pad2)
- D53 pad 1: D8 -> D5
- D53 pad 2: Net-(D10-Pad2) -> Net-(D17-Pad2)
- D54 pad 1: D9 -> D5
- D54 pad 2: Net-(D10-Pad2) -> Net-(D18-Pad2)
- D55 pad 1: D7 -> D6
- D55 pad 2: Net-(D18-Pad2) -> Net-(D10-Pad2)
- D56 pad 1: D8 -> D6
- D56 pad 2: Net-(D18-Pad2) -> Net-(D1-Pad2)
- D57 pad 1: D9 -> D6
- D57 pad 2: Net-(D18-Pad2) -> Net-(D11-Pad2)
- D58 pad 1: D7 -> D6
- D58 pad 2: Net-(D26-Pad2) -> Net-(D12-Pad2)
- D59 pad 1: D8 -> D6
- D59 pad 2: Net-(D26-Pad2) -> Net-(D13-Pad2)
- D6 pad 1: D4 -> D0
- D6 pad 2: Net-(D1-Pad2) -> Net-(D15-Pad2)
- D60 pad 1: D9 -> D6
- D60 pad 2: Net-(D26-Pad2) -> Net-(D14-Pad2)
- D61 pad 2: Net-(D34-Pad2) -> Net-(D16-Pad2)
- D62 pad 1: D7 -> D6
- D62 pad 2: Net-(D34-Pad2) -> Net-(D17-Pad2)
- D63 pad 1: D8 -> D6
- D63 pad 2: Net-(D34-Pad2) -> Net-(D18-Pad2)
- D64 pad 1: D9 -> D7
- D64 pad 2: Net-(D34-Pad2) -> Net-(D10-Pad2)
- D65 pad 1: D5 -> D7
- D65 pad 2: Net-(D17-Pad2) -> Net-(D1-Pad2)
- D66 pad 2: Net-(D17-Pad2) -> Net-(D11-Pad2)
- D67 pad 1: D8 -> D7
- D67 pad 2: Net-(D17-Pad2) -> Net-(D12-Pad2)
- D68 pad 1: D9 -> D7
- D68 pad 2: Net-(D17-Pad2) -> Net-(D13-Pad2)
- D69 pad 1: D5 -> D7
- D69 pad 2: Net-(D43-Pad2) -> Net-(D14-Pad2)
- D7 pad 1: D5 -> D0
- D7 pad 2: Net-(D1-Pad2) -> Net-(D16-Pad2)
- D70 pad 1: D6 -> D7
- D70 pad 2: (no net) -> Net-(D15-Pad2)
- D71 pad 1: D8 -> D7
- D71 pad 2: Net-(D43-Pad2) -> Net-(D17-Pad2)
- D72 pad 1: D9 -> D7
- D72 pad 2: Net-(D43-Pad2) -> Net-(D18-Pad2)
- D73 pad 1: D0 -> D8
- D73 pad 2: Net-(D73-Pad2) -> Net-(D10-Pad2)
- D74 pad 1: D1 -> D8
- D74 pad 2: Net-(D73-Pad2) -> Net-(D1-Pad2)
- D75 pad 1: D2 -> D8
- D75 pad 2: Net-(D73-Pad2) -> Net-(D11-Pad2)
- D76 pad 1: D3 -> D8
- D76 pad 2: Net-(D73-Pad2) -> Net-(D12-Pad2)
- D77 pad 1: D4 -> D8
- D77 pad 2: Net-(D73-Pad2) -> Net-(D13-Pad2)
- D78 pad 1: D5 -> D8
- D78 pad 2: Net-(D73-Pad2) -> Net-(D14-Pad2)
- D79 pad 1: D6 -> D8
- D79 pad 2: (no net) -> Net-(D15-Pad2)
- D8 pad 1: D6 -> D0
- D8 pad 2: Net-(D1-Pad2) -> Net-(D17-Pad2)
- D80 pad 1: D7 -> D8
- D80 pad 2: Net-(D73-Pad2) -> Net-(D16-Pad2)
- D81 pad 1: D9 -> D8
- D81 pad 2: Net-(D73-Pad2) -> Net-(D18-Pad2)
- D82 pad 1: D0 -> D9
- D82 pad 2: Net-(D82-Pad2) -> Net-(D10-Pad2)
- D83 pad 1: D1 -> D9
- D83 pad 2: Net-(D82-Pad2) -> Net-(D1-Pad2)
- D84 pad 1: D2 -> D9
- D84 pad 2: Net-(D82-Pad2) -> Net-(D11-Pad2)
- D85 pad 1: D3 -> D9
- D85 pad 2: Net-(D82-Pad2) -> Net-(D12-Pad2)
- D86 pad 1: D4 -> D9
- D86 pad 2: Net-(D82-Pad2) -> Net-(D13-Pad2)
- D87 pad 1: D5 -> D9
- D87 pad 2: Net-(D82-Pad2) -> Net-(D14-Pad2)
- D88 pad 1: D6 -> D9
- D88 pad 2: (no net) -> Net-(D15-Pad2)
- D89 pad 1: D7 -> D9
- D89 pad 2: Net-(D82-Pad2) -> Net-(D16-Pad2)
- D9 pad 2: Net-(D17-Pad2) -> Net-(D18-Pad2)
- D90 pad 1: D8 -> D9
- D90 pad 2: Net-(D82-Pad2) -> Net-(D17-Pad2)
- R1 pad 1: Net-(D1-Pad2) -> Net-(D10-Pad2)
- R10 pad 1: Net-(D82-Pad2) -> Net-(D18-Pad2)
- R2 pad 1: Net-(D12-Pad2) -> Net-(D1-Pad2)
- R3 pad 1: Net-(D10-Pad2) -> Net-(D11-Pad2)
- R4 pad 1: Net-(D18-Pad2) -> Net-(D12-Pad2)
- R5 pad 1: Net-(D26-Pad2) -> Net-(D13-Pad2)
- R6 pad 1: Net-(D34-Pad2) -> Net-(D14-Pad2)
- R7 pad 1: Net-(D17-Pad2) -> Net-(D15-Pad2)
- R8 pad 1: Net-(D43-Pad2) -> Net-(D16-Pad2)
- R9 pad 1: Net-(D73-Pad2) -> Net-(D17-Pad2)
- SW1 pad 1: Net-(SW1-Pad1) -> GND
- SW1 pad 2: GND -> Net-(SW1-Pad2)
- SW2 pad 1: GND -> Net-(SW2-Pad1)
- SW2 pad 2: Net-(SW2-Pad2) -> GND
Routing:
- net (no net): track 54.7 -> 0.00 mm, vias 5 -> 0
- net D5: track 34.2 -> 0.00 mm, vias 7 -> 0
- net D6: track 32.6 -> 0.00 mm, vias 3 -> 0
- net D2: track 28.6 -> 0.00 mm, vias 3 -> 0
- net D0: track 25.4 -> 0.00 mm, vias 2 -> 0
- net Net-(D12-Pad2): track 25.3 -> 0.00 mm, vias 4 -> 0
- net D3: track 25.2 -> 0.00 mm, vias 3 -> 0
- net Net-(D10-Pad2): track 23.9 -> 0.00 mm, vias 4 -> 0
- net D4: track 23.9 -> 0.00 mm, vias 3 -> 0
- net D1: track 23.6 -> 0.00 mm, vias 3 -> 0
- net Net-(D18-Pad2): track 21.8 -> 0.00 mm, vias 4 -> 0
- net Net-(D26-Pad2): track 21.4 -> 0.00 mm, vias 5 -> 0
- net Net-(D1-Pad2): track 21.2 -> 0.00 mm, vias 1 -> 0
- net Net-(D43-Pad2): track 16.0 -> 0.00 mm, vias 5 -> 0
- net Net-(D34-Pad2): track 15.8 -> 0.00 mm, vias 5 -> 0
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- removed copper zone on F.Cu, net +5V
- removed copper zone on B.Cu, net GND
Other:
- board outline removed
- net class 0.25 removed
- net class 6 mil removed
- net class Default: clearance 0.1 -> 0.2; trace_width 0.1 -> 0.25; via_dia 0.6 -> 0.8; via_drill 0.2 -> 0.4
- net class PCBWAY removed
- rule pad_to_mask_clearance: 0.05 -> 0
- rule trace_clearance: 0.1 -> 0.2
- rule trace_min: 0.1 -> 0.2
- rule via_min_drill: 0.2 -> 0.3

Commit message: First version layout
Parts:
- added J1: USB_B_Micro, Connectors:USB_Micro-B, F.Cu at (102.8, 89.5)
- moved U1 89.3 mm to (121.8, 83.2)
- moved BZ1 56.7 mm to (132.5, 85.2), turned to 270 degrees
- moved SW1 41.4 mm to (115.0, 95.0), turned to 180 degrees
- moved SW2 40.2 mm to (132.5, 95.0), turned to 180 degrees
- moved D19 39.0 mm to (111.2, 65.0), turned to 270 degrees
- moved SW3 38.6 mm to (150.0, 95.0), turned to 180 degrees
- moved D1 38.0 mm to (111.2, 59.0), turned to 270 degrees
- moved D62 37.5 mm to (151.2, 62.0), turned to 270 degrees
- moved D53 37.3 mm to (151.2, 59.0), turned to 270 degrees
- moved D46 36.1 mm to (133.8, 59.0), turned to 270 degrees
- moved D5 35.4 mm to (121.2, 59.0), turned to 270 degrees
- moved D6 35.4 mm to (123.8, 59.0), turned to 270 degrees
- moved D61 35.1 mm to (148.8, 62.0), turned to 270 degrees
- moved D2 34.3 mm to (113.8, 59.0), turned to 270 degrees
- moved D4 34.1 mm to (118.8, 59.0), turned to 270 degrees
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Connections:
- SW2 pad 1: Net-(SW2-Pad1) -> GND
- SW2 pad 2: GND -> Net-(SW2-Pad2)
- U1 pad 13: Net-(SW2-Pad1) -> Net-(SW3-Pad2)
- U1 pad 2: Net-(SW3-Pad2) -> Net-(SW1-Pad2)
- U1 pad 3: Net-(SW1-Pad2) -> Net-(SW2-Pad2)
Routing:
- net Net-(D10-Pad2): track 0.00 -> 132.2 mm, vias 0 -> 10
- net D5: track 0.00 -> 108.8 mm, vias 0 -> 4
- net Net-(D14-Pad2): track 0.00 -> 98.0 mm, vias 0 -> 10
- net D6: track 0.00 -> 97.9 mm, vias 0 -> 4
- net D7: track 0.00 -> 87.5 mm, vias 0 -> 4
- net D8: track 0.00 -> 79.3 mm, vias 0 -> 4
- net D9: track 0.00 -> 74.3 mm, vias 0 -> 4
- net Net-(D17-Pad2): track 0.00 -> 69.5 mm, vias 0 -> 12
- net Net-(D16-Pad2): track 0.00 -> 68.3 mm, vias 0 -> 12
- net Net-(D15-Pad2): track 0.00 -> 67.1 mm, vias 0 -> 12
- net Net-(D13-Pad2): track 0.00 -> 65.9 mm, vias 0 -> 10
- net Net-(D1-Pad2): track 0.00 -> 65.4 mm, vias 0 -> 10
- net D3: track 0.00 -> 64.9 mm, vias 0 -> 4
- net Net-(D12-Pad2): track 0.00 -> 63.9 mm, vias 0 -> 10
- net D4: track 0.00 -> 63.8 mm, vias 0 -> 4
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- added copper zone on F.Cu, net +5V
- added copper zone on B.Cu, net GND
Other:
- board outline added: 65 x 45 mm
- net class Default: clearance 0.2 -> 0.15; trace_width 0.25 -> 0.15
- rule trace_clearance: 0.2 -> 0.15
- rule trace_min: 0.2 -> 0.15

Commit message: Last update Oyvind
Parts:
- added C1: 0.1µF, Capacitors_SMD:C_0402, F.Cu at (121.0, 79.5)
- added C2: 1µF, Capacitors_SMD:C_0402, F.Cu at (122.2, 79.5)
Connections:
- J1 pad 2: Net-(J1-Pad2) -> (no net)
- J1 pad 3: Net-(J1-Pad3) -> (no net)
- J1 pad 4: Net-(J1-Pad4) -> (no net)
Routing:
- net RESET: track 45.4 -> 52.7 mm
- net +5V: track 1.48 -> 5.31 mm
- net GND: track 34.2 -> 36.6 mm, vias 6 -> 7
