File: Reference-designs/Attiny-2313/B-timer/B-timer.sch (KiCad schematic (older format))
At the start: 106 parts, among them J1 Conn_02x03_Odd_Even, SW1 SW_Push, SW2 SW_Push, SW3 SW_Push, U2 ATTINY2313-20MU

Commit message: Added a Bitraf library
Parts:
- added R?: R, symbol device:R
- R1: symbol device1:R -> device:R
Changed lines of the file:
@@
 EESchema Schematic File Version 4
-LIBS:B-timer-cache
 EELAYER 26 0
 EELAYER END
@@
 $EndComp
 $Comp
-L device1:R R1
+L device:R R1
 U 1 1 5A7CEE4F
 P 1450 1200
@@
 Wire Wire Line
 	6650 3800 6800 3800
+$Comp
+L device:R R?
+U 1 1 5BC0DDE6
+P 100 200
+F 0 "R?" H 170 246 50  0000 L CNN
+F 1 "R" H 170 155 50  0000 L CNN
+F 2 "" V 30  200 50  0001 C CNN
+F 3 "" H 100 200 50  0001 C CNN
+	1    100  200
+	1    0    0    -1
+$EndComp
 $EndSCHEMATC

Commit message: Update version
Parts:
- removed R?: R, symbol device:R
- added J1: USB_B_Micro, symbol Connector:USB_B_Micro
- BZ1: footprint (none) -> Buzzers_Beepers:Buzzer_Murata_PKMCS0909E4000-R1; symbol device1:Buzzer -> Device:Buzzer
- D1: renamed from D2; footprint Bitraf:LED_0402 -> LEDs:LED_0603; symbol device1:LED -> Device:LED
- D10: renamed from D3; footprint Bitraf:LED_0402 -> LEDs:LED_0603; symbol device1:LED -> Device:LED
- D11, D33: footprint Bitraf:LED_0402 -> LEDs:LED_0603; symbol device1:LED -> Device:LED
- D12: renamed from D19; footprint Bitraf:LED_0402 -> LEDs:LED_0603; symbol device1:LED -> Device:LED
- D13: renamed from D27; footprint Bitraf:LED_0402 -> LEDs:LED_0603; symbol device1:LED -> Device:LED
- D14: renamed from D35; footprint Bitraf:LED_0402 -> LEDs:LED_0603; symbol device1:LED -> Device:LED
- D15: renamed from D17; footprint Bitraf:LED_0402 -> LEDs:LED_0603; symbol device1:LED -> Device:LED
- D16: renamed from D44; footprint Bitraf:LED_0402 -> LEDs:LED_0603; symbol device1:LED -> Device:LED
- D17: renamed from D74; footprint Bitraf:LED_0402 -> LEDs:LED_0603; symbol device1:LED -> Device:LED
- D18: renamed from D83; footprint Bitraf:LED_0402 -> LEDs:LED_0603; symbol device1:LED -> Device:LED
- D19: renamed from D4; footprint Bitraf:LED_0402 -> LEDs:LED_0603; symbol device1:LED -> Device:LED
- D2: renamed from D10; footprint Bitraf:LED_0402 -> LEDs:LED_0603; symbol device1:LED -> Device:LED
- D20: renamed from D12; footprint Bitraf:LED_0402 -> LEDs:LED_0603; symbol device1:LED -> Device:LED
- D21: renamed from D20; footprint Bitraf:LED_0402 -> LEDs:LED_0603; symbol device1:LED -> Device:LED
- D22: renamed from D28; footprint Bitraf:LED_0402 -> LEDs:LED_0603; symbol device1:LED -> Device:LED
- D23: renamed from D36; footprint Bitraf:LED_0402 -> LEDs:LED_0603; symbol device1:LED -> Device:LED
- D24: renamed from D25; footprint Bitraf:LED_0402 -> LEDs:LED_0603; symbol device1:LED -> Device:LED
- D25: renamed from D45; footprint Bitraf:LED_0402 -> LEDs:LED_0603; symbol device1:LED -> Device:LED
- D26: renamed from D75; footprint Bitraf:LED_0402 -> LEDs:LED_0603; symbol device1:LED -> Device:LED
- D27: renamed from D84; footprint Bitraf:LED_0402 -> LEDs:LED_0603; symbol device1:LED -> Device:LED
- D28: renamed from D5; footprint Bitraf:LED_0402 -> LEDs:LED_0603; symbol device1:LED -> Device:LED
- D29: renamed from D13; footprint Bitraf:LED_0402 -> LEDs:LED_0603; symbol device1:LED -> Device:LED
- D3: renamed from D18; footprint Bitraf:LED_0402 -> LEDs:LED_0603; symbol device1:LED -> Device:LED
- D30: renamed from D21; footprint Bitraf:LED_0402 -> LEDs:LED_0603; symbol device1:LED -> Device:LED
- D31: renamed from D29; footprint Bitraf:LED_0402 -> LEDs:LED_0603; symbol device1:LED -> Device:LED
- D32: renamed from D37; footprint Bitraf:LED_0402 -> LEDs:LED_0603; symbol device1:LED -> Device:LED
- D34: renamed from D46; footprint Bitraf:LED_0402 -> LEDs:LED_0603; symbol device1:LED -> Device:LED
- D35: renamed from D76; footprint Bitraf:LED_0402 -> LEDs:LED_0603; symbol device1:LED -> Device:LED
- D36: renamed from D85; footprint Bitraf:LED_0402 -> LEDs:LED_0603; symbol device1:LED -> Device:LED
- D37: renamed from D6; footprint Bitraf:LED_0402 -> LEDs:LED_0603; symbol device1:LED -> Device:LED
- D38: renamed from D14; footprint Bitraf:LED_0402 -> LEDs:LED_0603; symbol device1:LED -> Device:LED
- D39: renamed from D22; footprint Bitraf:LED_0402 -> LEDs:LED_0603; symbol device1:LED -> Device:LED
- D4: renamed from D26; footprint Bitraf:LED_0402 -> LEDs:LED_0603; symbol device1:LED -> Device:LED
- D40: renamed from D30; footprint Bitraf:LED_0402 -> LEDs:LED_0603; symbol device1:LED -> Device:LED
- D41: renamed from D38; footprint Bitraf:LED_0402 -> LEDs:LED_0603; symbol device1:LED -> Device:LED
- D42: renamed from D41; footprint Bitraf:LED_0402 -> LEDs:LED_0603; symbol device1:LED -> Device:LED
- D43: renamed from D47; footprint Bitraf:LED_0402 -> LEDs:LED_0603; symbol device1:LED -> Device:LED
- D44: renamed from D77; footprint Bitraf:LED_0402 -> LEDs:LED_0603; symbol device1:LED -> Device:LED
- D45: renamed from D86; footprint Bitraf:LED_0402 -> LEDs:LED_0603; symbol device1:LED -> Device:LED
- D46: renamed from D7; footprint Bitraf:LED_0402 -> LEDs:LED_0603; symbol device1:LED -> Device:LED
- D47: renamed from D15; footprint Bitraf:LED_0402 -> LEDs:LED_0603; symbol device1:LED -> Device:LED
- D48: renamed from D23; footprint Bitraf:LED_0402 -> LEDs:LED_0603; symbol device1:LED -> Device:LED
- D49: renamed from D31; footprint Bitraf:LED_0402 -> LEDs:LED_0603; symbol device1:LED -> Device:LED
- D5: renamed from D34; footprint Bitraf:LED_0402 -> LEDs:LED_0603; symbol device1:LED -> Device:LED
- D50: renamed from D39; footprint Bitraf:LED_0402 -> LEDs:LED_0603; symbol device1:LED -> Device:LED
- D51: renamed from D65; footprint Bitraf:LED_0402 -> LEDs:LED_0603; symbol device1:LED -> Device:LED
- D52: renamed from D69; footprint Bitraf:LED_0402 -> LEDs:LED_0603; symbol device1:LED -> Device:LED
- D53: renamed from D78; footprint Bitraf:LED_0402 -> LEDs:LED_0603; symbol device1:LED -> Device:LED
- D54: renamed from D87; footprint Bitraf:LED_0402 -> LEDs:LED_0603; symbol device1:LED -> Device:LED
- D55: renamed from D8; footprint Bitraf:LED_0402 -> LEDs:LED_0603; symbol device1:LED -> Device:LED
- D56: renamed from D16; footprint Bitraf:LED_0402 -> LEDs:LED_0603; symbol device1:LED -> Device:LED
- D57: renamed from D24; footprint Bitraf:LED_0402 -> LEDs:LED_0603; symbol device1:LED -> Device:LED
- D58: renamed from D32; footprint Bitraf:LED_0402 -> LEDs:LED_0603; symbol device1:LED -> Device:LED
- D59: renamed from D40; footprint Bitraf:LED_0402 -> LEDs:LED_0603; symbol device1:LED -> Device:LED
- D6: renamed from D9; footprint Bitraf:LED_0402 -> LEDs:LED_0603; symbol device1:LED -> Device:LED
- D60: renamed from D61; footprint Bitraf:LED_0402 -> LEDs:LED_0603; symbol device1:LED -> Device:LED
- D61: renamed from D70; footprint Bitraf:LED_0402 -> LEDs:LED_0603; symbol device1:LED -> Device:LED
- D62: renamed from D79; footprint Bitraf:LED_0402 -> LEDs:LED_0603; symbol device1:LED -> Device:LED
- D63: renamed from D88; footprint Bitraf:LED_0402 -> LEDs:LED_0603; symbol device1:LED -> Device:LED
- D64: renamed from D1; footprint Bitraf:LED_0402 -> LEDs:LED_0603; symbol device1:LED -> Device:LED
- D65: renamed from D49; footprint Bitraf:LED_0402 -> LEDs:LED_0603; symbol device1:LED -> Device:LED
- D66: renamed from D52; footprint Bitraf:LED_0402 -> LEDs:LED_0603; symbol device1:LED -> Device:LED
- D67: renamed from D55; footprint Bitraf:LED_0402 -> LEDs:LED_0603; symbol device1:LED -> Device:LED
- D68: renamed from D58; footprint Bitraf:LED_0402 -> LEDs:LED_0603; symbol device1:LED -> Device:LED
- D69: renamed from D62; footprint Bitraf:LED_0402 -> LEDs:LED_0603; symbol device1:LED -> Device:LED
- D7: renamed from D43; footprint Bitraf:LED_0402 -> LEDs:LED_0603; symbol device1:LED -> Device:LED
- D70: renamed from D66; footprint Bitraf:LED_0402 -> LEDs:LED_0603; symbol device1:LED -> Device:LED
- D71: renamed from D80; footprint Bitraf:LED_0402 -> LEDs:LED_0603; symbol device1:LED -> Device:LED
- D72: renamed from D89; footprint Bitraf:LED_0402 -> LEDs:LED_0603; symbol device1:LED -> Device:LED
- D73: renamed from D42; footprint Bitraf:LED_0402 -> LEDs:LED_0603; symbol device1:LED -> Device:LED
- D74: renamed from D50; footprint Bitraf:LED_0402 -> LEDs:LED_0603; symbol device1:LED -> Device:LED
- D75: renamed from D53; footprint Bitraf:LED_0402 -> LEDs:LED_0603; symbol device1:LED -> Device:LED
- D76: renamed from D56; footprint Bitraf:LED_0402 -> LEDs:LED_0603; symbol device1:LED -> Device:LED
- D77: renamed from D59; footprint Bitraf:LED_0402 -> LEDs:LED_0603; symbol device1:LED -> Device:LED
- D78: renamed from D63; footprint Bitraf:LED_0402 -> LEDs:LED_0603; symbol device1:LED -> Device:LED
- D79: renamed from D67; footprint Bitraf:LED_0402 -> LEDs:LED_0603; symbol device1:LED -> Device:LED
- D8: renamed from D73; footprint Bitraf:LED_0402 -> LEDs:LED_0603; symbol device1:LED -> Device:LED
- D80: renamed from D71; footprint Bitraf:LED_0402 -> LEDs:LED_0603; symbol device1:LED -> Device:LED
- D81: renamed from D90; footprint Bitraf:LED_0402 -> LEDs:LED_0603; symbol device1:LED -> Device:LED
- D82: renamed from D48; footprint Bitraf:LED_0402 -> LEDs:LED_0603; symbol device1:LED -> Device:LED
- D83: renamed from D51; footprint Bitraf:LED_0402 -> LEDs:LED_0603; symbol device1:LED -> Device:LED
- D84: renamed from D54; footprint Bitraf:LED_0402 -> LEDs:LED_0603; symbol device1:LED -> Device:LED
- D85: renamed from D57; footprint Bitraf:LED_0402 -> LEDs:LED_0603; symbol device1:LED -> Device:LED
- D86: renamed from D60; footprint Bitraf:LED_0402 -> LEDs:LED_0603; symbol device1:LED -> Device:LED
- D87: renamed from D64; footprint Bitraf:LED_0402 -> LEDs:LED_0603; symbol device1:LED -> Device:LED
- D88: renamed from D68; footprint Bitraf:LED_0402 -> LEDs:LED_0603; symbol device1:LED -> Device:LED
- D89: renamed from D72; footprint Bitraf:LED_0402 -> LEDs:LED_0603; symbol device1:LED -> Device:LED
- D9: renamed from D82; footprint Bitraf:LED_0402 -> LEDs:LED_0603; symbol device1:LED -> Device:LED
- D90: renamed from D81; footprint Bitraf:LED_0402 -> LEDs:LED_0603; symbol device1:LED -> Device:LED
- J2: renamed from J1; footprint (none) -> Pin_Headers:Pin_Header_Straight_2x03_Pitch2.54mm_SMD; symbol conn:Conn_02x03_Odd_Even -> Connector_Generic:Conn_02x03_Odd_Even
- R1: footprint Bitraf:R_0402 -> Resistors_SMD:R_0402; symbol device:R -> Device:R
- R10, R2, R3, R4, R5, R6, R7, R8, R9: footprint Bitraf:R_0402 -> Resistors_SMD:R_0402; symbol device1:R -> Device:R
- SW1: renamed from SW2; footprint Bitraf:PTS_540 -> Buttons_Switches_SMD:SW_SPST_B3S-1000; symbol switches1:SW_Push -> Switch:SW_Push
- SW2: renamed from SW1; footprint Bitraf:PTS_540 -> Buttons_Switches_SMD:SW_SPST_B3S-1000; symbol switches1:SW_Push -> Switch:SW_Push
- SW3: footprint Bitraf:PTS_540 -> Buttons_Switches_SMD:SW_SPST_B3S-1000; symbol switches1:SW_Push -> Switch:SW_Push
- U1: renamed from U2; symbol atmel1:ATTINY2313-20MU -> MCU_Microchip_ATtiny:ATtiny2313-20MU
Connections:
- wire segments 526 -> 541
- no-connect marks 0 -> 3

Commit message: First version layout
Parts:
- J1: footprint (none) -> Connectors:USB_Micro-B
- renumbered SW3 to SW1, SW1 to SW2, SW2 to SW3
Changed lines of the file:
@@
 D6
 $Comp
-L Switch:SW_Push SW2
+L Switch:SW_Push SW3
 U 1 1 5A7F71BF
 P 10150 3600
-F 0 "SW2" H 10200 3700 50  0000 L CNN
+F 0 "SW3" H 10200 3700 50  0000 L CNN
 F 1 "SW_Push" H 10150 3540 50  0000 C CNN
 F 2 "Buttons_Switches_SMD:SW_SPST_B3S-1000" H 10150 3800 50  0001 C CNN
@@
 F 4 "PTS645SM43SMTR92 LFS" H 10150 3600 50  0001 C CNN "MPN"
 	1    10150 3600
-	1    0    0    -1
+	-1   0    0    -1
 $EndComp
 $Comp
@@
 	8450 3000 8450 2650
 $Comp
-L Switch:SW_Push SW3
+L Switch:SW_Push SW1
 U 1 1 5BBE28E4
 P 7350 3700
-F 0 "SW3" H 7050 3750 50  0000 L CNN
+F 0 "SW1" H 7050 3750 50  0000 L CNN
 F 1 "SW_Push" H 7350 3640 50  0001 C CNN
 F 2 "Buttons_Switches_SMD:SW_SPST_B3S-1000" H 7350 3900 50  0001 C CNN
@@
 	9850 3850 9950 3850
 $Comp
-L Switch:SW_Push SW1
+L Switch:SW_Push SW2
 U 1 1 5BCC52DE
 P 7350 3500
-F 0 "SW1" H 7050 3550 50  0000 L CNN
+F 0 "SW2" H 7050 3550 50  0000 L CNN
 F 1 "SW_Push" H 7350 3440 50  0001 C CNN
 F 2 "Buttons_Switches_SMD:SW_SPST_B3S-1000" H 7350 3700 50  0001 C CNN
@@
 Wire Wire Line
 	9650 1750 10050 1750
-Wire Wire Line
-	10350 3600 10550 3600
 $Comp
 L power:GND #PWR09
@@
 	9050 3500 9300 3500
 Wire Wire Line
-	9050 3600 9950 3600
-Wire Wire Line
 	9050 3700 9850 3700
 Wire Wire Line
@@
 F 0 "J1" H 6705 1917 50  0000 C CNN
 F 1 "USB_B_Micro" H 6705 1826 50  0000 C CNN
-F 2 "" H 6800 1400 50  0001 C CNN
+F 2 "Connectors:USB_Micro-B" H 6800 1400 50  0001 C CNN
 F 3 "~" H 6800 1400 50  0001 C CNN
 	1    6650 1450
@@
 NoConn ~ 6950 1550
 NoConn ~ 6950 1650
+Wire Wire Line
+	9950 3600 9050 3600
+Wire Wire Line
+	10350 3600 10550 3600
 $EndSCHEMATC

Commit message: Last update Oyvind
Parts:
- added C1: 0.1µF, Capacitors_SMD:C_0402, symbol Device:C
- added C2: 1µF, Capacitors_SMD:C_0402, symbol Device:C
- SW2: MPN PTS645SM43SMTR92 LFS -> PTS645SM43SMTR92LFS
Connections:
- wire segments 541 -> 548
Changed lines of the file:
@@
 EESchema Schematic File Version 4
+LIBS:B-timer-cache
 EELAYER 26 0
 EELAYER END
@@
 P 8450 4100
 F 0 "U1" H 8450 5378 50  0000 C CNN
-F 1 "ATTINY2313-20MU" H 8450 5287 50  0000 C CNN
+F 1 "ATTINY2313-20MU" H 8900 5150 50  0000 C CNN
 F 2 "Bitraf:VQFN20-SMALL" H 8450 4100 50  0001 C CIN
 F 3 "http://www.atmel.com/Images/doc2543.pdf" H 8450 4100 50  0001 C CNN
@@
 L power:+5V #PWR05
 U 1 1 5B9AEBFD
-P 8450 2650
-F 0 "#PWR05" H 8450 2500 50  0001 C CNN
-F 1 "+5V" H 8450 2790 50  0000 C CNN
-F 2 "" H 8450 2650 50  0000 C CNN
-F 3 "" H 8450 2650 50  0000 C CNN
-	1    8450 2650
-	1    0    0    -1
-$EndComp
-Wire Wire Line
-	8450 3000 8450 2650
+P 8450 2050
+F 0 "#PWR05" H 8450 1900 50  0001 C CNN
+F 1 "+5V" H 8450 2190 50  0000 C CNN
+F 2 "" H 8450 2050 50  0000 C CNN
+F 3 "" H 8450 2050 50  0000 C CNN
+	1    8450 2050
+	1    0    0    -1
+$EndComp
 $Comp
 L Switch:SW_Push SW1
@@
 L Connector_Generic:Conn_02x03_Odd_Even J2
 U 1 1 5BC4BA6E
-P 9350 1850
-F 0 "J2" H 9400 2167 50  0000 C CNN
-F 1 "Conn_02x03_Odd_Even" H 9400 2076 50  0000 C CNN
-F 2 "Pin_Headers:Pin_Header_Straight_2x03_Pitch2.54mm_SMD" H 9350 1850 50  0001 C CNN
-F 3 "~" H 9350 1850 50  0001 C CNN
-	1    9350 1850
+P 9650 1300
+F 0 "J2" H 9700 1617 50  0000 C CNN
+F 1 "Conn_02x03_Odd_Even" H 9700 1526 50  0000 C CNN
+F 2 "Pin_Headers:Pin_Header_Straight_2x03_Pitch2.54mm_SMD" H 9650 1300 50  0001 C CNN
+F 3 "~" H 9650 1300 50  0001 C CNN
+	1    9650 1300
 	1    0    0    -1
 $EndComp
@@
 F 2 "Buttons_Switches_SMD:SW_SPST_B3S-1000" H 7350 3700 50  0001 C CNN
 F 3 "" H 7350 3700 50  0000 C CNN
-F 4 "PTS645SM43SMTR92 LFS" H 7350 3500 50  0001 C CNN "MPN"
+F 4 "PTS645SM43SMTR92LFS" H 7350 3500 50  0001 C CNN "MPN"
 	1    7350 3500
 	1    0    0    -1
@@
 $EndComp
 Wire Wire Line
-	9150 1750 8950 1750
-Wire Wire Line
-	9150 1850 8950 1850
-Wire Wire Line
-	9150 1950 8950 1950
-Wire Wire Line
-	9650 1850 9950 1850
-Text GLabel 8950 1750 0    50   Input ~ 0
+	9450 1200 9250 1200
+Wire Wire Line
+	9450 1300 9250 1300
+Wire Wire Line
+	9450 1400 9250 1400
+Wire Wire Line
+	9950 1300 10250 1300
+Text GLabel 9250 1200 0    50   Input ~ 0
 MISO
-Text GLabel 8950 1850 0    50   Input ~ 0
+Text GLabel 9250 1300 0    50   Input ~ 0
 SCK
-Text GLabel 8950 1950 0    50   Input ~ 0
+Text GLabel 9250 1400 0    50   Input ~ 0
 RESET
-Text GLabel 9950 1850 2    50   Input ~ 0
+Text GLabel 10250 1300 2    50   Input ~ 0
 MOSI
 $Comp
 L power:+5V #PWR02
 U 1 1 5D5A1E3F
-P 10050 1600
-F 0 "#PWR02" H 10050 1450 50  0001 C CNN
-F 1 "+5V" H 10050 1740 50  0000 C CNN
-F 2 "" H 10050 1600 50  0000 C CNN
-F 3 "" H 10050 1600 50  0000 C CNN
-	1    10050 1600
+P 10350 1050
+F 0 "#PWR02" H 10350 900 50  0001 C CNN
+F 1 "+5V" H 10350 1190 50  0000 C CNN
+F 2 "" H 10350 1050 50  0000 C CNN
+F 3 "" H 10350 1050 50  0000 C CNN
+	1    10350 1050
 	1    0    0    -1
 $EndComp
@@
 L power:GND #PWR04
 U 1 1 5D5A31C0
-P 10050 2050
-F 0 "#PWR04" H 10050 1800 50  0001 C CNN
-F 1 "GND" H 10055 1877 50  0000 C CNN
-F 2 "" H 10050 2050 50  0001 C CNN
-F 3 "" H 10050 2050 50  0001 C CNN
-	1    10050 2050
-	1    0    0    -1
-$EndComp
-Wire Wire Line
-	10050 1950 10050 2050
-Wire Wire Line
-	9650 1950 10050 1950
-Wire Wire Line
-	10050 1750 10050 1600
-Wire Wire Line
-	9650 1750 10050 1750
+P 10350 1500
+F 0 "#PWR04" H 10350 1250 50  0001 C CNN
+F 1 "GND" H 10355 1327 50  0000 C CNN
+F 2 "" H 10350 1500 50  0001 C CNN
+F 3 "" H 10350 1500 50  0001 C CNN
+	1    10350 1500
+	1    0    0    -1
+$EndComp
+Wire Wire Line
+	10350 1400 10350 1500
+Wire Wire Line
+	9950 1400 10350 1400
+Wire Wire Line
+	10350 1200 10350 1050
+Wire Wire Line
+	9950 1200 10350 1200
 $Comp
 L power:GND #PWR09
@@
 Wire Wire Line
 	10350 3600 10550 3600
+$Comp
+L Device:C C1
+U 1 1 5BCA4C5A
+P 7900 2450
+F 0 "C1" H 8015 2496 50  0000 L CNN
+F 1 "0.1µF" H 8015 2405 50  0000 L CNN
+F 2 "Capacitors_SMD:C_0402" H 7938 2300 50  0001 C CNN
+F 3 "~" H 7900 2450 50  0001 C CNN
+	1    7900 2450
+	1    0    0    -1
+$EndComp
+Wire Wire Line
+	8450 2050 8450 2250
+Wire Wire Line
+	7900 2300 7900 2250
+Wire Wire Line
+	7900 2250 8450 2250
+Connection ~ 8450 2250
+Wire Wire Line
+	8450 2250 8450 3000
+$Comp
+L Device:C C2
+U 1 1 5BEC3F45
+P 8950 2450
+F 0 "C2" H 9065 2496 50  0000 L CNN
+F 1 "1µF" H 9065 2405 50  0000 L CNN
+F 2 "Capacitors_SMD:C_0402" H 8988 2300 50  0001 C CNN
+F 3 "~" H 8950 2450 50  0001 C CNN
+	1    8950 2450
+	1    0    0    -1
+$EndComp
+Wire Wire Line
+	8950 2250 8950 2300
+$Comp
+L power:GND #PWR0101
+U 1 1 5BFD60E6
+P 7900 2650
+F 0 "#PWR0101" H 7900 2400 50  0001 C CNN
+F 1 "GND" H 7905 2477 50  0000 C CNN
+F 2 "" H 7900 2650 50  0001 C CNN
+F 3 "" H 7900 2650 50  0001 C CNN
+	1    7900 2650
+	1    0    0    -1
+$EndComp
+$Comp
+L power:GND #PWR0102
+U 1 1 5BFD6312
+P 8950 2650
+F 0 "#PWR0102" H 8950 2400 50  0001 C CNN
+F 1 "GND" H 8955 2477 50  0000 C CNN
+F 2 "" H 8950 2650 50  0001 C CNN
+F 3 "" H 8950 2650 50  0001 C CNN
+	1    8950 2650
+	1    0    0    -1
+$EndComp
+Wire Wire Line
+	8950 2650 8950 2600
+Wire Wire Line
+	7900 2650 7900 2600
+Wire Wire Line
+	8450 2250 8950 2250
 $EndSCHEMATC
